File: board/power-clock.kicad_sch (KiCad schematic)
At the start: 9 parts, among them SW1 RESET, Y1 12 MHz

Commit message: fill out most functionality - passes ERC
Parts:
- removed R1: 100K, Resistors_SMD:R_0805, symbol MOBO_SMD-rescue:R
- removed R5: 100, Resistors_SMD:R_0805, symbol MOBO_SMD-rescue:R
- removed R6: 10K, Resistors_SMD:R_0805, symbol MOBO_SMD-rescue:R
- added R1: 100, symbol Device:R
- added R2: 10K, symbol Device:R
- added R33: 100K, symbol Device:R
- D1: value RED -> GREEN
- renumbered C10 to C1, C3 to C2, C12 to C3
Connections:
- net +5V: now also R2.1, R33.1
- net GND: now also R1.2
- net HALT: now also R2.2
- net at D1.1 (K): now also R1.1
- net at Y1.1 (EN): now also R33.2
Other:
- moved on the sheet: C2
