File: board/board.kicad_pcb (KiCad board)
At the start: 4 copper layers, 257 x 201.5 mm, 138 parts, among them J1 Conn_ARM_JTAG_SWD_10, J2 KEYBOARD, J3 AdaFruit 4090 USB-C BOB, J4 MOUSE, J5 AudioJack3, J6 COMPOSITE, J7 Conn_02x32_Counter_Clockwise, J8 SD_Card_Receptacle, J9 FTDI serial, SW1 RESET, U1 MC68000P, U10 RAM 4 LO, U11 RAM 4 HI, U12 GLUE, U13 SN74LVC245APW, U14 LD1117V33, U15 LM358, U16 AT89x51xxP, U17 CPST, U18 74HC373, U19 74HC373, U2 ROM LO, U20 74HC165, U21 74HC165, U22 74HC373, U23 74HC373, U24 DA56-11SRWA, U3 ROM HI, U4 RAM 1 LO, U5 RAM 1 HI, U6 RAM 2 LO, U7 RAM 2 HI, U8 RAM 3 LO, U9 RAM 3 HI, Y1 14.318MHz, Y2 11.0592MHz, Y4 12MHz

Commit message: checkpoint
Parts:
- removed R17, R18, R19, R20, R21, R22, R23, R24, R25, R26, R27, R28, R29, R30, R31, R32: 330, Resistor_THT:R_Axial_DIN0207_L6.3mm_D2.5mm_P10.16mm_Horizontal
- removed R35, R37, R39, R41, R43, R45, R47, R49: 10K, Resistor_THT:R_Axial_DIN0207_L6.3mm_D2.5mm_P10.16mm_Horizontal
- removed R36, R38, R40, R42, R44, R46, R48, R50, R51: 20K, Resistor_THT:R_Axial_DIN0207_L6.3mm_D2.5mm_P10.16mm_Horizontal
- removed REF** (x4): MountingHole_3.2mm_M3_Pad, MountingHole:MountingHole_3.2mm_M3_Pad
- added H1: MountingHole_Pad, MountingHole:MountingHole_2.5mm_Pad, F.Cu at (105.8, 105.8)
- added H2: MountingHole_Pad, MountingHole:MountingHole_2.5mm_Pad, F.Cu at (346.2, 105.7)
- added H3: MountingHole_Pad, MountingHole:MountingHole_2.5mm_Pad, F.Cu at (345.9, 266.3)
- added H4: MountingHole_Pad, MountingHole:MountingHole_2.5mm_Pad, F.Cu at (105.5, 266.4)
- added H5: MountingHole_Pad, MountingHole:MountingHole_2.5mm_Pad, F.Cu at (105.5, 119.2)
- added H6: MountingHole_Pad, MountingHole:MountingHole_2.5mm_Pad, F.Cu at (235.5, 119.2)
- added H7: MountingHole_Pad, MountingHole:MountingHole_2.5mm_Pad, F.Cu at (235.5, 239.2)
- added H8: MountingHole_Pad, MountingHole:MountingHole_2.5mm_Pad, F.Cu at (105.5, 239.2)
- added H9: MountingHole_Pad, MountingHole:MountingHole_2.5mm_Pad, F.Cu at (226.9, 190.7)
- added LS1: Speaker, Buzzer_Beeper:MagneticBuzzer_StarMicronics_QMX, F.Cu at (185.0, 243.9)
- added R59: 100, Resistor_THT:R_Axial_DIN0207_L6.3mm_D2.5mm_P10.16mm_Horizontal, F.Cu at (174.3, 245.7)
- added R60: 4610X-R2R-103LF, board:BO_4610X, F.Cu at (288.8, 140.0)
- added RN1: 330, Package_DIP:DIP-16_W7.62mm, F.Cu at (217.2, 248.5)
- added RN2: 330, Package_DIP:DIP-16_W7.62mm, F.Cu at (266.2, 248.7)
- J1: value Conn_ARM_JTAG_SWD_10 -> Conn_01x05_Pin; footprint Connector_PinHeader_1.27mm:PinHeader_2x05_P1.27mm_Vertical -> Connector_PinHeader_2.54mm:PinHeader_1x05_P2.54mm_Vertical
- J9: footprint Connector_PinHeader_2.54mm:PinHeader_1x06_P2.54mm_Vertical -> Connector_PinHeader_2.54mm:PinHeader_1x06_P2.54mm_Horizontal
- U20, U21: footprint Package_DIP:DIP-20_W7.62mm -> Package_DIP:DIP-16_W7.62mm
- moved J1 113.5 mm to (130.0, 135.9)
- moved U2 105.5 mm to (226.4, 145.1)
- moved U3 102.7 mm to (226.1, 198.0)
- moved C6 96.6 mm to (234.1, 138.1), turned to 0 degrees
- moved C7 94.3 mm to (235.3, 190.8), turned to 0 degrees
- moved U17 75.9 mm to (203.3, 154.2), turned to 0 degrees
- moved R12 69.3 mm to (169.2, 162.7)
- moved Y1 65.2 mm to (178.5, 156.5), turned to 90 degrees
- moved C13 64.7 mm to (320.5, 147.7)
- moved C11 64.1 mm to (295.1, 147.7)
- moved C14 64.1 mm to (320.5, 195.8)
- moved C12 64.0 mm to (295.2, 195.8)
- moved C9 63.9 mm to (269.8, 195.8)
- moved C10 63.8 mm to (269.8, 147.7)
- moved C15 63.6 mm to (345.8, 147.7)
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Connections:
- J1 pad 1: +5V -> GND
- J1 pad 2: JTAG_TMS -> JTAG_TCK
- J1 pad 3: GND -> JTAG_TDI
- J1 pad 4: JTAG_TCK -> JTAG_TDO
- J1 pad 5: GND -> JTAG_TMS
- J8 pad 12: unconnected-(J8-SHELL1-Pad12) -> GND
- J8 pad 13: unconnected-(J8-SHELL2-Pad13) -> GND
- U12 pad 48: A1 -> BOOT_BEEP
- U12 pad 49: A2 -> ~{R}/W
- U12 pad 50: A3 -> ~{HALT}
- U12 pad 51: ~{R}/W -> A2
- U12 pad 52: ~{HALT} -> A1
- U12 pad 54: unconnected-(U12-I/O-Pad54) -> A3
- U12 pad 55: unconnected-(U12-I/O-Pad55) -> A15
- U12 pad 56: unconnected-(U12-I/O-Pad56) -> A16
- U12 pad 57: unconnected-(U12-I/O-Pad57) -> A17
- U12 pad 58: unconnected-(U12-I/O-Pad58) -> A18
- U12 pad 60: CPST_START_FIELD -> A19
- U12 pad 61: AUDIO_LE -> CPST_SELECT
- U12 pad 69: unconnected-(U12-I/O-Pad69) -> CPST_START_FIELD
- U12 pad 84: GND -> ~{CPST_DTACK}
- U13 pad 5: unconnected-(U13-A4-Pad5) -> GND
- U13 pad 6: unconnected-(U13-A5-Pad6) -> GND
- U13 pad 7: unconnected-(U13-A6-Pad7) -> GND
- U13 pad 8: unconnected-(U13-A7-Pad8) -> GND
- U13 pad 9: unconnected-(U13-A8-Pad9) -> GND
- U17 pad 30: AUDIO_LE -> ~{CPST_SELECT}
- U17 pad 37: unconnected-(U17-I/O-Pad37) -> ~{CPST_DTACK}
- U24 pad 13: Net-(U24-DIG2_CA) -> +5V
- U24 pad 14: Net-(U24-DIG1_CA) -> +5V
- U24 pad 4: +5V -> Net-(RN1-R8.2)
- U24 pad 9: +5V -> Net-(RN2-R4.1)
Routing:
- net SYSCLK: track 0.00 -> 187.8 mm, vias 0 -> 4
- net ~{RESET}: track 0.00 -> 116.3 mm, vias 0 -> 4
- net ~{VIDEO_IACK}: track 0.00 -> 111.7 mm, vias 0 -> 2
- net +3V3: track 0.00 -> 110.4 mm
- net CPST_CLK: track 0.00 -> 97.9 mm, vias 0 -> 1
- net A22: track 0.00 -> 68.3 mm, vias 0 -> 2
- net A23: track 0.00 -> 64.6 mm, vias 0 -> 2
- net D6: track 0.00 -> 57.0 mm, vias 0 -> 2
- net D8: track 0.00 -> 54.8 mm, vias 0 -> 2
- net Net-(U21-Q7): track 0.00 -> 54.3 mm, vias 0 -> 1
- net D10: track 0.00 -> 53.8 mm, vias 0 -> 2
- net D7: track 0.00 -> 53.6 mm, vias 0 -> 2
- net D5: track 0.00 -> 53.2 mm, vias 0 -> 2
- net ~{IPL0}: track 0.00 -> 53.1 mm, vias 0 -> 2
- net D9: track 0.00 -> 51.6 mm, vias 0 -> 2
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- added copper zone on In2.Cu, net +5V
- added copper zone on In1.Cu, net GND
Other:
- board size 257 x 201.5 mm -> 252.1 x 172.4 mm
- board text added: "Approx FT232H BOB footprint"

Commit message: checkpoint
Parts:
- moved C5 2.34 mm to (160.0, 186.7)
Connections:
- U12 pad 61: CPST_SELECT -> ~{CPST_SELECT}
- U17 pad 1: DEBUG_IN -> GND
Routing:
- net DEBUG_IN: track 0.00 -> 87.9 mm, vias 0 -> 1
- net DEBUG_OUT: track 0.00 -> 54.0 mm, vias 0 -> 1
- net SD_CS_3V3: track 6.91 -> 35.4 mm
- net SD_DI_3V3: track 6.40 -> 32.6 mm
- net SD_SCK_3V3: track 6.40 -> 27.9 mm
- net SD_3V3OE: track 0.00 -> 13.8 mm, vias 0 -> 2
- net ~{IPL0}: track 53.1 -> 49.8 mm, vias 2 -> 3
- net GND: track 8.57 -> 6.21 mm, vias 1 -> 0
- net A22: track 68.3 -> 66.9 mm
- net +3V3: track 110.4 -> 109.6 mm

Commit message: checkpoint - maybe unfinishable
Parts:
- added R17: 10K, Resistor_THT:R_Axial_DIN0207_L6.3mm_D2.5mm_P10.16mm_Horizontal, F.Cu at (160.0, 218.7)
- added R18: 10K, Resistor_THT:R_Axial_DIN0207_L6.3mm_D2.5mm_P10.16mm_Horizontal, F.Cu at (160.0, 222.8)
- added R19: 10K, Resistor_THT:R_Axial_DIN0207_L6.3mm_D2.5mm_P10.16mm_Horizontal, F.Cu at (170.3, 226.9)
- moved C6 7.93 mm to (241.4, 141.2), turned to 180 degrees
- moved C7 6.46 mm to (241.3, 193.2), turned to 180 degrees
- moved C20 3.21 mm to (156.1, 240.8)
- moved R10 3.21 mm to (152.3, 235.6)
- moved R11 3.21 mm to (159.8, 235.6)
- moved R7 3.21 mm to (148.6, 235.6)
- moved R9 3.21 mm to (163.6, 235.6)
- moved C26 2.41 mm to (260.7, 111.1), turned to 180 degrees
- moved Y2 0.13 mm to (328.1, 133.2)
Connections:
- J7 pad 32: unconnected-(J7-Pin_32-Pad32) -> VIDEO_PRESENT
- U12 pad 55: A15 -> VIDEO_PRESENT
Routing:
- net A2: track 0.00 -> 487.7 mm, vias 0 -> 9
- net A3: track 0.00 -> 474.7 mm, vias 0 -> 12
- net A12: track 0.00 -> 467.6 mm, vias 0 -> 9
- net A14: track 0.00 -> 461.6 mm, vias 0 -> 6
- net A9: track 0.00 -> 455.6 mm, vias 0 -> 7
- net A10: track 0.00 -> 453.2 mm, vias 0 -> 7
- net A11: track 0.00 -> 450.0 mm, vias 0 -> 7
- net A13: track 0.00 -> 447.0 mm, vias 0 -> 9
- net A1: track 0.00 -> 444.3 mm, vias 0 -> 8
- net A16: track 0.00 -> 430.4 mm, vias 0 -> 5
- net A15: track 0.00 -> 428.6 mm, vias 0 -> 6
- net A4: track 0.00 -> 427.4 mm, vias 0 -> 6
- net A19: track 0.00 -> 425.9 mm, vias 0 -> 11
- net ~{R}/W: track 0.00 -> 425.8 mm, vias 0 -> 5
- net A8: track 0.00 -> 423.8 mm, vias 0 -> 8
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
Commit message: checkpoint before reordering 1508 inputs
Parts:
- removed H5, H8: MountingHole_Pad, MountingHole:MountingHole_2.5mm_Pad
- H1, H2, H3, H4, H6, H7, H9: footprint MountingHole:MountingHole_2.5mm_Pad -> MountingHole:MountingHole_2.5mm_Pad_Via
- J7: value Conn_02x32_Counter_Clockwise -> Expansion Bus; footprint Connector_PinHeader_2.54mm:PinHeader_2x32_P2.54mm_Vertical -> Connector_PinHeader_2.54mm:PinHeader_2x36_P2.54mm_Vertical
- moved TP1 195.4 mm to (308.4, 108.2)
- moved TP2 195.4 mm to (308.4, 118.8)
- moved LS1 132.7 mm to (316.4, 261.8)
- moved R59 132.7 mm to (305.8, 263.6)
- moved J1 96.8 mm to (217.3, 177.7), turned to 180 degrees
- moved U13 73.2 mm to (189.6, 279.6), turned to 180 degrees
- moved C18 72.9 mm to (193.3, 277.2), turned to 90 degrees
- moved R8 69.1 mm to (178.2, 280.0), turned to 90 degrees
- moved C36 57.6 mm to (216.7, 254.7)
- moved C30 54.5 mm to (185.9, 197.2), turned to 180 degrees
- moved C31 51.9 mm to (128.9, 139.9)
- moved C32 51.9 mm to (128.5, 119.7)
- moved C33 51.9 mm to (158.0, 120.3)
- moved C34 51.9 mm to (159.6, 136.1)
- moved U18 51.9 mm to (140.1, 140.5)
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Connections:
- net SD_CS_3V3 renamed ~{SD_CS_3V3}
- net SD_DI_3V3 renamed SPI_DI_3V3
- net SD_DI_5V renamed SPI_DI_5V
- net SD_DO_3V3 renamed SPI_DO_3V3
- net SD_SCK_3V3 renamed SPI_SCK_3V3
- net SD_SCK_5V renamed SPI_SCK_5V
- C18 pad 1: +5V -> +3V3
- C20 pad 1: +5V -> +3V3
- J7 pad 1: SYSCLK -> +3V3
- J7 pad 10: D3 -> D8
- J7 pad 11: D4 -> D0
- J7 pad 12: D5 -> D9
- J7 pad 13: D6 -> ~{AS}
- J7 pad 14: D7 -> D10
- J7 pad 15: D8 -> ~{UDS}
- J7 pad 16: D9 -> D11
- J7 pad 17: D10 -> ~{LDS}
- J7 pad 18: D11 -> D12
- J7 pad 19: D12 -> R/~{W}
- J7 pad 2: ~{LDS} -> +3V3
- J7 pad 21: D14 -> ~{R}/W
- J7 pad 22: D15 -> D14
- J7 pad 23: ~{VIDEO_SELECT} -> ~{BG}
- J7 pad 24: ~{VIDEO_DTACK} -> D15
- J7 pad 25: ~{VIDEO_IRQ} -> ~{BGACK}
- J7 pad 26: ~{DTACK} -> GND
- J7 pad 27: ~{BERR} -> ~{BR}
- J7 pad 28: ~{BR} -> A23
- J7 pad 29: ~{BG} -> +5V
- J7 pad 3: ~{UDS} -> D4
- J7 pad 30: ~{BGACK} -> A22
- J7 pad 31: ~{VIDEO_IACK} -> SYSCLK
- J7 pad 32: VIDEO_PRESENT -> A21
- J7 pad 33: unconnected-(J7-Pin_33-Pad33) -> GND
- J7 pad 34: ~{RESET} -> +5V
- J7 pad 36: ~{IPL0} -> A20
- J7 pad 37: ~{IPL1} -> ~{RESET}
- J7 pad 38: ~{IPL2} -> A19
- J7 pad 39: ~{FC0} -> ~{BERR}
- J7 pad 4: ~{AS} -> D5
- J7 pad 40: ~{FC1} -> A18
- J7 pad 41: ~{FC2} -> ~{IPL2}
- J7 pad 42: A23 -> A17
- J7 pad 43: A22 -> ~{IPL1}
- J7 pad 44: A21 -> A16
- J7 pad 45: A20 -> ~{IPL0}
- J7 pad 46: A19 -> A15
- J7 pad 47: A18 -> ~{FC2}
- J7 pad 48: A17 -> A14
- J7 pad 49: A16 -> ~{FC1}
- J7 pad 5: R/~{W} -> D3
- J7 pad 50: A15 -> A13
- J7 pad 51: A14 -> ~{FC0}
- J7 pad 52: A13 -> A12
- J7 pad 53: A12 -> A1
- J7 pad 55: A10 -> A2
- J7 pad 56: A9 -> A10
- J7 pad 57: A8 -> A3
- J7 pad 58: A7 -> A9
- J7 pad 59: A6 -> A4
- J7 pad 6: ~{R}/W -> D6
- J7 pad 60: A5 -> A8
- J7 pad 61: A4 -> ~{VIDEO_SELECT}
- J7 pad 62: A3 -> A7
- J7 pad 63: A2 -> ~{VIDEO_DTACK}
- J7 pad 64: A1 -> A6
- J7 pad 7: D0 -> D2
- J7 pad 8: D1 -> D7
- J7 pad 9: D2 -> D1
Routing:
- net A2: track 487.7 -> 0.00 mm, vias 9 -> 0
- net A3: track 474.7 -> 0.00 mm, vias 12 -> 0
- net A12: track 467.6 -> 0.00 mm, vias 9 -> 0
- net A14: track 461.6 -> 0.00 mm, vias 6 -> 0
- net A9: track 455.6 -> 0.00 mm, vias 7 -> 0
- net A10: track 453.2 -> 0.00 mm, vias 7 -> 0
- net A11: track 450.0 -> 0.00 mm, vias 7 -> 0
- net A13: track 447.0 -> 0.00 mm, vias 9 -> 0
- net A1: track 444.3 -> 0.00 mm, vias 8 -> 0
- net A16: track 430.4 -> 0.00 mm, vias 5 -> 0
- net A15: track 428.6 -> 0.00 mm, vias 6 -> 0
- net A4: track 427.4 -> 0.00 mm, vias 6 -> 0
- net A19: track 425.9 -> 0.00 mm, vias 11 -> 0
- net ~{R}/W: track 425.8 -> 0.00 mm, vias 5 -> 0
- net A8: track 423.8 -> 0.00 mm, vias 8 -> 0
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Other:
- board size 252.1 x 172.4 mm -> 240.4 x 183.4 mm
- board text removed: "Approx FT232H BOB footprint"

Commit message: checkpoint
Parts:
- moved J9 214.0 mm to (114.0, 139.0), turned to 180 degrees
- moved C31 207.9 mm to (336.8, 135.2)
- moved U18 207.9 mm to (347.9, 135.8)
- moved C32 207.9 mm to (336.3, 115.0)
- moved U20 207.9 mm to (324.4, 115.8)
- moved TP1 183.5 mm to (126.0, 128.6), turned to 180 degrees
- moved TP2 182.4 mm to (126.0, 118.0), turned to 180 degrees
- moved C30 147.1 mm to (331.4, 218.7)
- moved U17 147.1 mm to (337.6, 180.5)
- moved R12 147.1 mm to (348.1, 171.2)
- moved Y1 147.1 mm to (341.9, 161.9)
- moved U21 146.9 mm to (293.5, 117.0)
- moved C33 146.9 mm to (304.8, 116.0)
- moved C34 146.9 mm to (306.3, 131.8)
- moved U19 146.9 mm to (317.5, 136.2)
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Connections:
- net Net-(U21-Q7) renamed CPST_PIXEL
- U12 pad 1: DEBUG_IN -> CPST_START_FIELD
- U12 pad 10: A21 -> ~{WRITE_LO}
- U12 pad 11: A22 -> ~{WRITE_HI}
- U12 pad 12: A23 -> ~{IO_SELECT}
- U12 pad 15: ~{ROM_SELECT} -> ~{VIDEO_SELECT}
- U12 pad 16: ~{RAM_SELECT_1} -> ~{IO_DTACK}
- U12 pad 17: ~{RAM_SELECT_2} -> ~{VIDEO_DTACK}
- U12 pad 18: ~{RAM_SELECT_3} -> ~{IO_IRQ}
- U12 pad 2: ~{RESET} -> VIDEO_PRESENT
- U12 pad 20: ~{RAM_SELECT_4} -> ~{VIDEO_IRQ}
- U12 pad 21: ~{WRITE_LO} -> ~{IO_IACK}
- U12 pad 22: ~{WRITE_HI} -> D5
- U12 pad 24: ~{IO_SELECT} -> D3
- U12 pad 25: ~{VIDEO_SELECT} -> D7
- U12 pad 27: ~{IO_DTACK} -> D1
- U12 pad 28: ~{VIDEO_DTACK} -> ~{UDS}
- U12 pad 29: ~{IO_IRQ} -> ~{LDS}
- U12 pad 30: ~{VIDEO_IRQ} -> ~{DTACK}
- U12 pad 31: ~{IO_IACK} -> A23
- U12 pad 33: ~{DTACK} -> A20
- U12 pad 34: ~{BERR} -> SYSCLK
- U12 pad 35: ~{IPL0} -> A19
- U12 pad 36: ~{IPL1} -> ~{HALT}
- U12 pad 37: ~{IPL2} -> ~{RESET}
- U12 pad 39: ~{FC0} -> A17
- U12 pad 4: ~{LDS} -> ~{ROM_SELECT}
- U12 pad 40: ~{FC1} -> A18
- U12 pad 41: ~{FC2} -> A16
- U12 pad 44: DEBUG_OUT -> ~{BERR}
- U12 pad 45: DBGLOLED_LE -> ~{IPL1}
- U12 pad 46: DBGHILED_LE -> ~{IPL2}
- U12 pad 48: BOOT_BEEP -> ~{IPL0}
- U12 pad 49: ~{R}/W -> ~{FC1}
- U12 pad 5: ~{UDS} -> ~{RAM_SELECT_1}
- U12 pad 50: ~{HALT} -> ~{FC2}
- U12 pad 51: A2 -> A1
- U12 pad 52: A1 -> ~{FC0}
- U12 pad 55: VIDEO_PRESENT -> A2
- U12 pad 56: A16 -> A21
- U12 pad 57: A17 -> A22
- U12 pad 58: A18 -> R/~{W}
- U12 pad 6: R/~{W} -> ~{RAM_SELECT_2}
- U12 pad 60: A19 -> ~{AS}
- U12 pad 61: ~{CPST_SELECT} -> D0
- U12 pad 63: SPI_DO_3V3 -> D2
- U12 pad 64: SPI_DI_5V -> D6
- U12 pad 65: SPI_SCK_5V -> D4
- U12 pad 67: SD_3V3OE -> DEBUG_OUT
- U12 pad 68: SD_CS_5V -> DBGLOLED_LE
- U12 pad 69: CPST_START_FIELD -> DBGHILED_LE
- U12 pad 70: ~{VIDEO_IACK} -> BOOT_BEEP
- U12 pad 73: D0 -> ~{R}/W
- U12 pad 74: D1 -> ~{CPST_SELECT}
- U12 pad 75: D2 -> ~{VIDEO_IACK}
- U12 pad 76: D3 -> SPI_DO_3V3
- U12 pad 77: D4 -> SPI_DI_5V
- U12 pad 79: D5 -> SPI_SCK_5V
- U12 pad 8: ~{AS} -> ~{RAM_SELECT_3}
- U12 pad 80: D6 -> SD_3V3OE
- U12 pad 81: D7 -> SD_CS_5V
- U12 pad 83: SYSCLK -> DEBUG_IN
- U12 pad 9: A20 -> ~{RAM_SELECT_4}
- U17 pad 10: A21 -> ~{CPST_SYNC}
- U17 pad 11: A22 -> D5
- U17 pad 12: A23 -> D4
- U17 pad 15: D8 -> D3
- U17 pad 16: D9 -> D8
- U17 pad 17: D10 -> D2
- U17 pad 18: D11 -> D0
- U17 pad 20: D12 -> D11
- U17 pad 21: D13 -> ~{AS}
- U17 pad 22: D14 -> ~{UDS}
- U17 pad 24: D15 -> D13
- U17 pad 25: unconnected-(U17-I/O-Pad25) -> R/~{W}
- U17 pad 27: unconnected-(U17-I/O-Pad27) -> D15
- U17 pad 28: unconnected-(U17-I/O-Pad28) -> A21
- U17 pad 29: unconnected-(U17-I/O-Pad29) -> SYSCLK
- U17 pad 30: ~{CPST_SELECT} -> A19
- U17 pad 31: CPST_START_FIELD -> A18
- U17 pad 33: CPST_FILL -> A14
- U17 pad 34: CPST_LE -> A15
- U17 pad 35: ~{CPST_SYNC} -> A12
- U17 pad 36: ~{CPST_PL} -> A13
- U17 pad 37: ~{CPST_DTACK} -> A11
- U17 pad 39: ~{FC0} -> A10
- U17 pad 4: ~{LDS} -> ~{CPST_SELECT}
- U17 pad 40: ~{FC1} -> ~{FC2}
- U17 pad 41: ~{FC2} -> ~{FC1}
- U17 pad 44: ~{BGACK} -> A9
- U17 pad 45: ~{BG} -> A8
- U17 pad 46: ~{BR} -> ~{FC0}
- U17 pad 5: ~{UDS} -> CPST_START_FIELD
- U17 pad 50: A3 -> A7
- U17 pad 51: A4 -> A3
- U17 pad 52: A5 -> A6
- U17 pad 54: A6 -> A4
- U17 pad 55: A7 -> A5
- U17 pad 56: A8 -> A16
- U17 pad 57: A9 -> A17
- U17 pad 58: A10 -> A20
- U17 pad 6: R/~{W} -> unconnected-(U17-I/O-Pad6)
- U17 pad 60: A11 -> A22
- U17 pad 61: A12 -> A23
- U17 pad 63: A13 -> D14
- U17 pad 64: A14 -> ~{LDS}
- U17 pad 65: A15 -> D12
- U17 pad 67: A16 -> D10
- U17 pad 68: A17 -> D1
- U17 pad 69: A18 -> D9
- U17 pad 70: A19 -> D7
- U17 pad 73: D0 -> D6
- U17 pad 74: D1 -> ~{BGACK}
- U17 pad 75: D2 -> ~{BG}
- U17 pad 76: D3 -> ~{BR}
- U17 pad 77: D4 -> ~{CPST_PL}
- U17 pad 79: D5 -> ~{CPST_DTACK}
- U17 pad 8: ~{AS} -> CPST_FILL
- U17 pad 80: D6 -> unconnected-(U17-I/O-Pad80)
- U17 pad 81: D7 -> unconnected-(U17-I/O/GCLK3-Pad81)
- U17 pad 83: SYSCLK -> unconnected-(U17-INPUT/GCLK1-Pad83)
- U17 pad 9: A20 -> CPST_LE
Routing:
- net ~{CPST_SYNC}: track 0.00 -> 131.4 mm, vias 0 -> 1
- net +3V3: track 0.00 -> 96.7 mm
- net A4: track 0.00 -> 95.3 mm, vias 0 -> 2
- net SYSCLK: track 0.00 -> 94.8 mm, vias 0 -> 3
- net A3: track 0.00 -> 92.1 mm, vias 0 -> 1
- net ~{IPL0}: track 0.00 -> 89.3 mm, vias 0 -> 2
- net A2: track 0.00 -> 82.8 mm, vias 0 -> 1
- net MOUSE_CLK: track 0.00 -> 82.2 mm, vias 0 -> 2
- net ~{IPL1}: track 0.00 -> 78.2 mm, vias 0 -> 3
- net ~{FC0}: track 0.00 -> 76.4 mm, vias 0 -> 1
- net A1: track 0.00 -> 75.8 mm, vias 0 -> 2
- net A15: track 0.00 -> 74.1 mm, vias 0 -> 2
- net A14: track 0.00 -> 73.2 mm
- net UART_RX: track 0.00 -> 72.8 mm, vias 0 -> 1
- net ~{IPL2}: track 0.00 -> 71.8 mm, vias 0 -> 4
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Other:
- board size 240.4 x 183.4 mm -> 260.6 x 176.9 mm

Commit message: checkpoint before CPST shrink
Routing:
- net ~{BERR}: track 52.2 -> 55.2 mm, vias 0 -> 1
- net ~{IPL2}: track 71.8 -> 70.3 mm, vias 4 -> 2
- net ~{RESET}: track 68.9 -> 68.0 mm
- net A21: track 57.6 -> 56.9 mm
- net A15: track 74.1 -> 73.4 mm
- net SYSCLK: track 94.8 -> 95.4 mm

Commit message: checkpoint before deleting composite video
Parts:
- removed C31, C32, C33, C34: 100nF, Capacitor_THT:C_Disc_D5.0mm_W2.5mm_P5.00mm
- removed U18, U19: 74HC373, Package_DIP:DIP-20_W7.62mm
- removed U20, U21: 74HC165, Package_DIP:DIP-16_W7.62mm
- added C27: 100nF, Capacitor_THT:C_Disc_D5.0mm_W2.5mm_P5.00mm, F.Cu at (325.4, 165.4)
- added J10: VGA, board:HD15-SN-24, F.Cu at (320.5, 100.1)
- added R20: 100K, Resistor_THT:R_Axial_DIN0207_L6.3mm_D2.5mm_P10.16mm_Horizontal, F.Cu at (346.6, 168.2)
- added R21: 270, Resistor_THT:R_Axial_DIN0207_L6.3mm_D2.5mm_P10.16mm_Horizontal, F.Cu at (333.1, 118.8)
- added R25: 270, Resistor_THT:R_Axial_DIN0207_L6.3mm_D2.5mm_P10.16mm_Horizontal, F.Cu at (324.7, 118.8)
- added R26: 560, Resistor_THT:R_Axial_DIN0207_L6.3mm_D2.5mm_P10.16mm_Horizontal, F.Cu at (320.5, 118.8)
- added R31: 270, Resistor_THT:R_Axial_DIN0207_L6.3mm_D2.5mm_P10.16mm_Horizontal, F.Cu at (312.0, 118.8)
- added R40: 150, Resistor_THT:R_Axial_DIN0207_L6.3mm_D2.5mm_P10.16mm_Horizontal, F.Cu at (328.9, 128.9)
- added R41: 150, Resistor_THT:R_Axial_DIN0207_L6.3mm_D2.5mm_P10.16mm_Horizontal, F.Cu at (316.2, 128.9)
- added R42: 150, Resistor_THT:R_Axial_DIN0207_L6.3mm_D2.5mm_P10.16mm_Horizontal, F.Cu at (307.8, 128.9)
- added Y3: 25.175MHz, Oscillator:Oscillator_DIP-8, F.Cu at (340.5, 159.5)
- U17: value CPST -> OBVID
- moved C16 22.5 mm to (325.6, 145.6)
- moved R12 22.5 mm to (346.7, 148.7)
- moved Y1 22.5 mm to (340.5, 139.4)
Connections:
- net CPST_START_FIELD renamed OBVID_FRAME
- net CPST_TDI renamed OBVID_TDI
- net ~{CPST_DTACK} renamed ~{OBVID_DTACK}
- net ~{CPST_SELECT} renamed ~{OBVID_SELECT}
- U17 pad 40: ~{FC2} -> unconnected-(U17-I/O-Pad40)
- U17 pad 41: ~{FC1} -> unconnected-(U17-I/O-Pad41)
- U17 pad 46: ~{FC0} -> VGA_HSYNC
- U17 pad 6: unconnected-(U17-I/O-Pad6) -> VGA_G0
- U17 pad 77: ~{CPST_PL} -> VGA_B0
- U17 pad 8: CPST_FILL -> VGA_G1
- U17 pad 80: unconnected-(U17-I/O-Pad80) -> CPST_PIXEL
- U17 pad 81: unconnected-(U17-I/O/GCLK3-Pad81) -> VGA_R0
- U17 pad 83: unconnected-(U17-INPUT/GCLK1-Pad83) -> VGA_CLK
- U17 pad 9: CPST_LE -> unconnected-(U17-I/O-Pad9)
Routing:
- net ~{CPST_SYNC}: track 131.4 -> 1.56 mm, vias 1 -> 0
- net CPST_FILL: track 55.2 -> 0.00 mm, vias 1 -> 0
- net CPST_CLK: track 0.00 -> 39.9 mm, vias 0 -> 1
- net CPST_PIXEL: track 39.2 -> 0.00 mm, vias 1 -> 0
- net ~{CPST_PL}: track 32.5 -> 0.00 mm
- net Net-(U20-Q7): track 31.9 -> 0.00 mm
- net CPST_LE: track 31.1 -> 0.00 mm
- net Net-(U18-O4): track 22.8 -> 0.00 mm, vias 2 -> 0
- net Net-(U18-O3): track 22.7 -> 0.00 mm, vias 2 -> 0
- net Net-(U19-O3): track 22.0 -> 0.00 mm, vias 2 -> 0
- net VGA_BLUE: track 0.00 -> 22.0 mm, vias 0 -> 1
- net VGA_GREEN: track 0.00 -> 20.9 mm
- net Net-(U19-O0): track 20.2 -> 0.00 mm, vias 2 -> 0
- net VGA_CLK: track 0.00 -> 20.1 mm, vias 0 -> 1
- net Net-(U18-O0): track 19.0 -> 0.00 mm, vias 2 -> 0
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
Commit message: checkpoint before compact flash
Parts:
- removed C27: 100nF, Capacitor_THT:C_Disc_D5.0mm_W2.5mm_P5.00mm
- removed J10: VGA, board:HD15-SN-24
- removed R20: 100K, Resistor_THT:R_Axial_DIN0207_L6.3mm_D2.5mm_P10.16mm_Horizontal
- removed R21, R25, R31: 270, Resistor_THT:R_Axial_DIN0207_L6.3mm_D2.5mm_P10.16mm_Horizontal
- removed R26: 560, Resistor_THT:R_Axial_DIN0207_L6.3mm_D2.5mm_P10.16mm_Horizontal
- removed R40, R41, R42: 150, Resistor_THT:R_Axial_DIN0207_L6.3mm_D2.5mm_P10.16mm_Horizontal
- removed Y3: 25.175MHz, Oscillator:Oscillator_DIP-8
- moved R12 80.4 mm to (285.0, 97.0), turned to 0 degrees
- moved C35 73.3 mm to (325.1, 163.5), turned to 90 degrees
- moved Y1 31.5 mm to (340.1, 170.9), turned to 90 degrees
- moved C16 20.2 mm to (319.1, 164.7)
- moved R16 18.7 mm to (285.0, 109.2), turned to 0 degrees
- moved J6 18.6 mm to (275.4, 104.0)
- moved R14 17.5 mm to (285.0, 101.1), turned to 0 degrees
- moved R15 6.52 mm to (285.0, 105.1), turned to 0 degrees
Connections:
- U17 pad 46: VGA_HSYNC -> unconnected-(U17-I/O-Pad46)
- U17 pad 6: VGA_G0 -> unconnected-(U17-I/O-Pad6)
- U17 pad 77: VGA_B0 -> unconnected-(U17-I/O-Pad77)
- U17 pad 8: VGA_G1 -> unconnected-(U17-I/O-Pad8)
- U17 pad 81: VGA_R0 -> unconnected-(U17-I/O/GCLK3-Pad81)
- U17 pad 83: VGA_CLK -> unconnected-(U17-INPUT/GCLK1-Pad83)
Routing:
- net CPST_CLK: track 39.9 -> 1.98 mm, vias 1 -> 0
- net VGA_BLUE: track 22.0 -> 0.00 mm, vias 1 -> 0
- net VGA_GREEN: track 20.9 -> 0.00 mm
- net VGA_CLK: track 20.1 -> 0.00 mm, vias 1 -> 0
- net VGA_RED: track 17.6 -> 0.00 mm
- net Net-(C35-Pad1): track 17.2 -> 0.00 mm
- net Net-(C35-Pad2): track 15.3 -> 0.00 mm, vias 1 -> 0
- net Net-(J6-In): track 10.5 -> 0.00 mm
- net Net-(Y3-EN): track 6.68 -> 0.00 mm
- net Net-(Y1-EN): track 6.58 -> 0.00 mm
- net ~{CPST_SYNC}: track 1.56 -> 0.00 mm
- net unconnected-(U17-INPUT/GCLK1-Pad83): track 0.00 -> 1.38 mm
