File: board/board.kicad_pcb (KiCad board)
At the start: 4 copper layers, 260.6 x 176.9 mm, 108 parts, among them J1 Conn_01x05_Pin, J2 KEYBOARD, J3 AdaFruit 4090 USB-C BOB, J4 MOUSE, J5 AudioJack3, J6 COMPOSITE, J7 Expansion Bus, J8 SD_Card_Receptacle, J9 FTDI serial, SW1 RESET, U1 MC68000P, U10 RAM 4 LO, U11 RAM 4 HI, U12 GLUE, U13 SN74LVC245APW, U14 LD1117V33, U15 LM358, U16 AT89x51xxP, U17 OBVID, U2 ROM LO, U22 74HC373, U23 74HC373, U24 DA56-11SRWA, U3 ROM HI, U4 RAM 1 LO, U5 RAM 1 HI, U6 RAM 2 LO, U7 RAM 2 HI, U8 RAM 3 LO, U9 RAM 3 HI, Y1 14.318MHz, Y2 11.0592MHz, Y4 12MHz

Commit message: CF card, composite, VGA
Parts:
- removed C18, C20: 100nF, Capacitor_THT:C_Disc_D5.0mm_W2.5mm_P5.00mm
- removed C19, C38: 10µF, Capacitor_THT:CP_Radial_D5.0mm_P2.50mm
- removed R10, R11, R7, R9: 68K, Resistor_THT:R_Axial_DIN0207_L6.3mm_D2.5mm_P10.16mm_Horizontal
- removed R8: 10K, Resistor_THT:R_Axial_DIN0207_L6.3mm_D2.5mm_P10.16mm_Horizontal
- removed U13: SN74LVC245APW, Package_DIP:DIP-20_W7.62mm
- removed U14: LD1117V33, Package_TO_SOT_THT:TO-220-3_Vertical
- added C27: 100nF, Capacitor_THT:C_Disc_D5.0mm_W2.5mm_P5.00mm, F.Cu at (345.8, 156.0)
- added J10: VGA, board:HD15-SN-24, F.Cu at (323.1, 100.3)
- added R20: 560, Resistor_THT:R_Axial_DIN0207_L6.3mm_D2.5mm_P10.16mm_Horizontal, F.Cu at (297.9, 130.8)
- added R21: 270, Resistor_THT:R_Axial_DIN0207_L6.3mm_D2.5mm_P10.16mm_Horizontal, F.Cu at (301.9, 130.8)
- added R22: 1100, Resistor_SMD:R_0603_1608Metric, F.Cu at (345.0, 147.4)
- added R23: 1100, Resistor_SMD:R_0603_1608Metric, F.Cu at (347.5, 147.4)
- added R25: 270, Resistor_THT:R_Axial_DIN0207_L6.3mm_D2.5mm_P10.16mm_Horizontal, F.Cu at (306.0, 130.8)
- added R26: 560, Resistor_THT:R_Axial_DIN0207_L6.3mm_D2.5mm_P10.16mm_Horizontal, F.Cu at (310.1, 130.8)
- added R31: 270, Resistor_THT:R_Axial_DIN0207_L6.3mm_D2.5mm_P10.16mm_Horizontal, F.Cu at (314.1, 130.8)
- added R40: 150, Resistor_THT:R_Axial_DIN0207_L6.3mm_D2.5mm_P10.16mm_Horizontal, F.Cu at (318.1, 130.8)
- added R41: 150, Resistor_THT:R_Axial_DIN0207_L6.3mm_D2.5mm_P10.16mm_Horizontal, F.Cu at (322.2, 130.8)
- added R42: 150, Resistor_THT:R_Axial_DIN0207_L6.3mm_D2.5mm_P10.16mm_Horizontal, F.Cu at (326.2, 130.8)
- added Y3: 25.175MHz, Oscillator:Oscillator_DIP-8, F.Cu at (340.4, 154.2)
- J8: value SD_Card_Receptacle -> CF Card; footprint board:10067847-001RLF -> board:SAMTEC_CFT-125-01-L-D-RA-01-SL
- R12: value 100K -> 560
- TP1: value Debug In -> TestPoint
- TP2: value Debug Out -> TestPoint
- moved TP2 67.3 mm to (180.4, 157.6), turned to 90 degrees
- moved TP1 52.6 mm to (170.0, 157.4), turned to 90 degrees
- moved R12 34.9 mm to (293.9, 130.8), turned to 90 degrees
- moved J8 10.3 mm to (154.0, 250.5)
Connections:
- net CPST_CLK renamed PIXEL_CLK
- J7 pad 1: +3V3 -> unconnected-(J7-Pin_1-Pad1)
- J7 pad 2: +3V3 -> unconnected-(J7-Pin_2-Pad2)
- J8 pad 10: unconnected-(J8-CARD_DETECT-Pad10) -> GND
- J8 pad 11: unconnected-(J8-WRITE_PROTECT-Pad11) -> GND
- J8 pad 13: GND -> +5V
- R12 pad 1: +5V -> VGA_BLUE
- R12 pad 2: Net-(Y1-EN) -> VGA_B0
- U12 pad 76: SPI_DO_3V3 -> ~{CF_CS0}
- U12 pad 77: SPI_DI_5V -> ~{CF_CS1}
- U12 pad 79: SPI_SCK_5V -> unconnected-(U12-I/O-Pad79)
- U12 pad 80: SD_3V3OE -> unconnected-(U12-I/O-Pad80)
- U12 pad 81: SD_CS_5V -> unconnected-(U12-I/O/GCLK3-Pad81)
- U17 pad 29: SYSCLK -> VGA_VSYNC
- U17 pad 4: ~{OBVID_SELECT} -> VGA_R0
- U17 pad 40: unconnected-(U17-I/O-Pad40) -> CPST_CLK_ENB
- U17 pad 41: unconnected-(U17-I/O-Pad41) -> VGA_CLK_ENB
- U17 pad 46: unconnected-(U17-I/O-Pad46) -> VGA_HSYNC
- U17 pad 6: unconnected-(U17-I/O-Pad6) -> VGA_R2
- U17 pad 74: ~{BGACK} -> VGA_B0
- U17 pad 75: ~{BG} -> VGA_B1
- U17 pad 76: ~{BR} -> VGA_G0
- U17 pad 77: unconnected-(U17-I/O-Pad77) -> VGA_G1
- U17 pad 8: unconnected-(U17-I/O-Pad8) -> VGA_R1
- U17 pad 81: unconnected-(U17-I/O/GCLK3-Pad81) -> VGA_G2
- U17 pad 83: unconnected-(U17-INPUT/GCLK1-Pad83) -> SYSCLK
- U17 pad 84: GND -> ~{OBVID_SELECT}
- U17 pad 9: unconnected-(U17-I/O-Pad9) -> VGA_R0
- Y1 pad 1: Net-(Y1-EN) -> CPST_CLK_ENB
Routing:
- net +3V3: track 96.7 -> 0.00 mm
- net SPI_SCK_3V3: track 67.5 -> 0.00 mm, vias 3 -> 0
- net SPI_DI_3V3: track 43.8 -> 0.00 mm, vias 3 -> 0
- net ~{SD_CS_3V3}: track 38.1 -> 0.00 mm, vias 3 -> 0
- net SPI_DO_3V3: track 23.2 -> 0.00 mm, vias 2 -> 0
- net SD_3V3OE: track 10.7 -> 0.00 mm, vias 1 -> 0
- net unconnected-(U17-INPUT/GCLK1-Pad83): track 1.38 -> 0.00 mm
- net SYSCLK: track 95.4 -> 96.8 mm
- net GND: vias 2 -> 0

Commit message: checkpoint
Parts:
- removed C37: 100nF, Capacitor_THT:C_Disc_D5.0mm_W2.5mm_P5.00mm
- removed H6, H7: MountingHole_Pad, MountingHole:MountingHole_2.5mm_Pad_Via
- removed J5: AudioJack3, Connector_Audio:Jack_3.5mm_CUI_SJ1-3523N_Horizontal
- removed R17, R18: 10K, Resistor_THT:R_Axial_DIN0207_L6.3mm_D2.5mm_P10.16mm_Horizontal
- removed RN1, RN2: 330, Package_DIP:DIP-16_W7.62mm
- removed U22: 74HC373, Package_DIP:DIP-20_W7.62mm
- removed U24: DA56-11SRWA, Display_7Segment:DA56-11SURKWA
- added C18: 100nF, Capacitor_THT:C_Disc_D5.0mm_W2.5mm_P5.00mm, F.Cu at (317.8, 254.4)
- added R7: 10K, Resistor_THT:R_Axial_DIN0207_L6.3mm_D2.5mm_P10.16mm_Horizontal, F.Cu at (222.7, 117.8)
- added R9: 10K, Resistor_THT:R_Axial_DIN0207_L6.3mm_D2.5mm_P10.16mm_Horizontal, F.Cu at (204.7, 126.9)
- added TP10: ~{UDS}, TestPoint:TestPoint_THTPad_D2.0mm_Drill1.0mm, F.Cu at (258.8, 265.9)
- added TP11: FC0, TestPoint:TestPoint_THTPad_D2.0mm_Drill1.0mm, F.Cu at (217.0, 272.6)
- added TP12: FC1, TestPoint:TestPoint_THTPad_D2.0mm_Drill1.0mm, F.Cu at (223.5, 272.6)
- added TP13: FC2, TestPoint:TestPoint_THTPad_D2.0mm_Drill1.0mm, F.Cu at (229.9, 272.6)
- added TP14: ~{ROM_SELECT}, TestPoint:TestPoint_THTPad_D2.0mm_Drill1.0mm, F.Cu at (236.3, 272.6)
- added TP15: ~{RAM_SELECT_1}, TestPoint:TestPoint_THTPad_D2.0mm_Drill1.0mm, F.Cu at (242.8, 272.6)
- added TP3: CLK, TestPoint:TestPoint_THTPad_D2.0mm_Drill1.0mm, F.Cu at (213.8, 265.9)
- added TP4: ~{RESET}, TestPoint:TestPoint_THTPad_D2.0mm_Drill1.0mm, F.Cu at (220.3, 265.9)
- added TP5: ~{HALT}, TestPoint:TestPoint_THTPad_D2.0mm_Drill1.0mm, F.Cu at (226.7, 265.9)
- added TP6: ~{AS}, TestPoint:TestPoint_THTPad_D2.0mm_Drill1.0mm, F.Cu at (233.1, 265.9)
- added TP7: ~{DTACK}, TestPoint:TestPoint_THTPad_D2.0mm_Drill1.0mm, F.Cu at (239.5, 265.9)
- added TP8: R/~{W}, TestPoint:TestPoint_THTPad_D2.0mm_Drill1.0mm, F.Cu at (246.0, 265.9)
- added TP9: ~{LDS}, TestPoint:TestPoint_THTPad_D2.0mm_Drill1.0mm, F.Cu at (252.4, 265.9)
- added U13: ENGINE, Package_LCC:PLCC-84_THT-Socket, F.Cu at (335.3, 218.1)
- J7: value Expansion Bus -> STEREO_OUT; footprint Connector_PinHeader_2.54mm:PinHeader_2x36_P2.54mm_Vertical -> board:SAMESKY_SJ3-35063B
- R22, R23: footprint Resistor_SMD:R_0603_1608Metric -> Resistor_THT:R_Axial_DIN0207_L6.3mm_D2.5mm_P10.16mm_Horizontal
- R59: value 100 -> 47
- TP1: value TestPoint -> Debug In
- TP2: value TestPoint -> Debug Out
- moved LS1 241.9 mm to (111.2, 127.1), turned to 0 degrees
- moved R59 230.8 mm to (109.3, 135.9), turned to 0 degrees
- moved TP1 139.5 mm to (249.2, 272.3)
- moved TP2 137.1 mm to (255.6, 272.3)
- moved C36 130.3 mm to (173.2, 125.4), turned to 0 degrees
- moved U23 116.1 mm to (173.9, 137.2), turned to -90 degrees
- moved J9 89.9 mm to (199.9, 112.5), turned to 90 degrees
- moved J7 78.5 mm to (172.2, 102.2), turned to 180 degrees
- moved C21 65.3 mm to (280.4, 118.5)
- moved C23 65.3 mm to (244.9, 118.0)
- moved U16 65.3 mm to (221.0, 136.8)
- moved C22 65.3 mm to (277.8, 135.3)
- moved Y2 65.3 mm to (278.8, 129.6)
- moved R12 60.9 mm to (352.7, 115.1), turned to -90 degrees
- moved C35 55.1 mm to (289.8, 121.0)
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Connections:
- net OBVID_FRAME renamed ~{OBVID_IRQ}
- net ~{OBVID_DTACK} renamed OBVID_STALL
- J7 pad 1: unconnected-(J7-Pin_1-Pad1) -> GND
- J7 pad 2: unconnected-(J7-Pin_2-Pad2) -> Net-(J7-Pad2)
- J7 pad 3: D4 -> Net-(J7-Pad3)
- J7 pad 4: D5 -> Net-(J7-Pad4)
- J8 pad 27: D11 -> unconnected-(J8-Pad27)
- J8 pad 28: D12 -> unconnected-(J8-Pad28)
- J8 pad 29: D13 -> unconnected-(J8-Pad29)
- J8 pad 30: D14 -> unconnected-(J8-Pad30)
- J8 pad 31: D15 -> unconnected-(J8-Pad31)
- J8 pad 47: D8 -> unconnected-(J8-Pad47)
- J8 pad 48: D9 -> unconnected-(J8-Pad48)
- J8 pad 49: D10 -> unconnected-(J8-Pad49)
- J8 pad S1: (no net) -> GND
- J8 pad S2: (no net) -> GND
- J8 pad S3: (no net) -> GND
- J8 pad S4: (no net) -> GND
- R19 pad 1: VIDEO_PRESENT -> Net-(U12-INPUT/OE2/GCLK2)
- R57 pad 1: Net-(J5-PadR) -> Net-(J7-Pad2)
- R58 pad 1: Net-(J5-PadT) -> Net-(J7-Pad3)
- R59 pad 2: BOOT_BEEP -> Net-(J7-Pad4)
- U1 pad 15: SYSCLK -> CPUCLK
- U1 pad 26: ~{FC2} -> FC2
- U1 pad 27: ~{FC1} -> FC1
- U1 pad 28: ~{FC0} -> FC0
- U10 pad 24: ~{R}/W -> GND
- U11 pad 24: ~{R}/W -> GND
- U12 pad 12: ~{IO_SELECT} -> ~{IO_SELECT_MOSI}
- U12 pad 15: ~{VIDEO_SELECT} -> ~{ENGINE_SELECT}
- U12 pad 16: ~{IO_DTACK} -> ~{IO_DTACK_MISO}
- U12 pad 17: ~{VIDEO_DTACK} -> ~{ENGINE_DTACK}
- U12 pad 2: VIDEO_PRESENT -> Net-(U12-INPUT/OE2/GCLK2)
- U12 pad 20: ~{VIDEO_IRQ} -> ~{ENGINE_IRQ}
- U12 pad 21: ~{IO_IACK} -> ~{IO_IACK_SCK}
- U12 pad 34: SYSCLK -> CPUCLK
- U12 pad 39: A17 -> ENGINE_TCK
- U12 pad 40: A18 -> ENGINE_TDI
- U12 pad 41: A16 -> ENGINE_TDO
- U12 pad 49: ~{FC1} -> FC1
- U12 pad 50: ~{FC2} -> FC2
- U12 pad 52: ~{FC0} -> FC0
- U12 pad 68: DBGLOLED_LE -> AUDIO_LE
- U12 pad 69: DBGHILED_LE -> IO_RESET
- U12 pad 70: BOOT_BEEP -> ENGINE_TMS
- U12 pad 75: ~{VIDEO_IACK} -> ~{ENGINE_IACK}
- U12 pad 79: unconnected-(U12-I/O-Pad79) -> A4
- U12 pad 80: unconnected-(U12-I/O-Pad80) -> A5
- U12 pad 81: unconnected-(U12-I/O/GCLK3-Pad81) -> A6
- U16 pad 1: AUDIO0 -> unconnected-(U16-P1.0-Pad1)
- U16 pad 12: KBD_CLK -> KBD_DATA
- U16 pad 13: MOUSE_CLK -> KBD_CLK
- U16 pad 14: KBD_DATA -> MOUSE_DATA
- U16 pad 15: MOUSE_DATA -> MOUSE_CLK
- U16 pad 2: AUDIO1 -> unconnected-(U16-P1.1-Pad2)
- U16 pad 25: ~{IO_SELECT} -> ~{IO_IRQ}
- U16 pad 26: ~{IO_IRQ} -> unconnected-(U16-P2.5/A13-Pad26)
- U16 pad 27: ~{IO_DTACK} -> unconnected-(U16-P2.6/A14-Pad27)
- U16 pad 28: ~{IO_IACK} -> unconnected-(U16-P2.7/A15-Pad28)
- U16 pad 3: AUDIO2 -> unconnected-(U16-P1.2-Pad3)
- U16 pad 4: AUDIO3 -> unconnected-(U16-P1.3-Pad4)
- U16 pad 5: AUDIO4 -> unconnected-(U16-P1.4-Pad5)
- U16 pad 6: AUDIO5 -> ~{IO_SELECT_MOSI}
- U16 pad 7: AUDIO6 -> ~{IO_DTACK_MISO}
- U16 pad 8: AUDIO7 -> ~{IO_IACK_SCK}
- U16 pad 9: ~{RESET} -> IO_RESET
- U17 pad 33: A14 -> ~{FC0}
- U17 pad 34: A15 -> ~{FC1}
- U17 pad 35: A12 -> ~{FC2}
- U17 pad 83: SYSCLK -> CPUCLK
- U23 pad 11: DBGHILED_LE -> AUDIO_LE
- U23 pad 12: Net-(RN1-R8.1) -> AUDIO4
- U23 pad 15: Net-(RN1-R3.1) -> AUDIO5
- U23 pad 16: Net-(RN1-R6.1) -> AUDIO6
- U23 pad 19: Net-(RN1-R1.1) -> AUDIO7
- U23 pad 2: Net-(RN1-R2.1) -> AUDIO0
- U23 pad 5: Net-(RN1-R4.1) -> AUDIO1
- U23 pad 6: Net-(RN1-R5.1) -> AUDIO2
- U23 pad 9: Net-(RN1-R7.1) -> AUDIO3
- U4 pad 24: ~{R}/W -> GND
- U5 pad 24: ~{R}/W -> GND
- U6 pad 24: ~{R}/W -> GND
- U7 pad 24: ~{R}/W -> GND
- U8 pad 24: ~{R}/W -> GND
- U9 pad 24: ~{R}/W -> GND
- Y4 pad 5: SYSCLK -> CPUCLK
Routing:
- net SYSCLK: track 96.8 -> 0.00 mm, vias 3 -> 0
- net A4: track 95.3 -> 0.00 mm, vias 2 -> 0
- net A3: track 92.1 -> 0.00 mm, vias 1 -> 0
- net ~{IPL0}: track 89.3 -> 0.00 mm, vias 2 -> 0
- net A2: track 82.8 -> 0.00 mm, vias 1 -> 0
- net MOUSE_CLK: track 82.2 -> 0.00 mm, vias 2 -> 0
- net ~{IPL1}: track 78.4 -> 0.00 mm, vias 3 -> 0
- net ~{FC0}: track 76.4 -> 0.00 mm, vias 1 -> 0
- net A1: track 75.8 -> 0.00 mm, vias 2 -> 0
- net A15: track 73.4 -> 0.00 mm, vias 2 -> 0
- net A14: track 73.1 -> 0.00 mm
- net UART_RX: track 72.8 -> 0.00 mm, vias 1 -> 0
- net ~{FC1}: track 71.4 -> 0.00 mm, vias 2 -> 0
- net ~{FC2}: track 70.6 -> 0.00 mm, vias 1 -> 0
- net ~{IPL2}: track 70.3 -> 0.00 mm, vias 2 -> 0
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Other:
- board size 260.6 x 176.9 mm -> 260.6 x 185.6 mm
