File: board/debug-led.kicad_sch (KiCad schematic)
At the start: 21 parts, among them U22 74HC373, U23 74HC373, U24 DA56-11SRWA

Commit message: design draft complete, added footprints
Parts:
- C36, C37: footprint (none) -> Capacitor_THT:C_Disc_D5.0mm_W2.5mm_P5.00mm
- R17, R18, R19, R20, R21, R22, R23, R24, R25, R26, R27, R28, R29, R30, R31, R32: footprint (none) -> Resistor_THT:R_Axial_DIN0207_L6.3mm_D2.5mm_P10.16mm_Horizontal
- U22, U23: footprint (none) -> Package_DIP:DIP-20_W7.62mm
Connections:
- net +5V: now also U24.4 (DP1), U24.9 (DP2)
- net GND: no longer U24.4 (DP1), U24.9 (DP2)
Changed lines of the file:
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@@
 	(wire
 		(pts
-			(xy 93.98 109.22) (xy 76.2 109.22)
+			(xy 93.98 109.22) (xy 78.74 109.22)
+		)
+		(stroke
+			(width 0)
+			(type default)
+		)
+	)
+	(wire
+		(pts
+			(xy 78.74 87.63) (xy 78.74 109.22)
 		)
 		(stroke
@@
 	(wire
 		(pts
-			(xy 135.89 109.22) (xy 135.89 116.84)
-		)
-		(stroke
-			(width 0)
-			(type default)
-		)
-	)
-	(wire
-		(pts
 			(xy 63.5 72.39) (xy 63.5 104.14)
 		)
@@
 	(wire
 		(pts
+			(xy 135.89 87.63) (xy 135.89 109.22)
+		)
+		(stroke
+			(width 0)
+			(type default)
+		)
+	)
+	(wire
+		(pts
 			(xy 95.25 165.1) (xy 92.71 165.1)
 		)
@@
 		(pts
 			(xy 142.24 27.94) (xy 142.24 78.74)
-		)
-		(stroke
-			(width 0)
-			(type default)
-		)
-	)
-	(wire
-		(pts
-			(xy 76.2 109.22) (xy 76.2 116.84)
 		)
 		(stroke
@@
 			)
 		)
-		(property "Footprint" ""
+		(property "Footprint" "Resistor_THT:R_Axial_DIN0207_L6.3mm_D2.5mm_P10.16mm_Horizontal"
 			(at 90.17 93.218 90)
 			(effects
@@
 			)
 		)
-		(property "Footprint" ""
+		(property "Footprint" "Resistor_THT:R_Axial_DIN0207_L6.3mm_D2.5mm_P10.16mm_Horizontal"
 			(at 128.27 93.218 90)
 			(effects
@@
 	(symbol
 		(lib_id "power:GND")
-		(at 135.89 116.84 0)
-		(unit 1)
-		(exclude_from_sim no)
-		(in_bom yes)
-		(on_board yes)
-		(dnp no)
-		(fields_autoplaced yes)
-		(property "Reference" "#PWR0134"
-			(at 135.89 123.19 0)
-			(effects
-				(font
-					(size 1.27 1.27)
-				)
-				(hide yes)
-			)
-		)
-		(property "Value" "GND"
-			(at 135.89 121.92 0)
-			(effects
-				(font
-					(size 1.27 1.27)
-				)
-			)
-		)
-		(property "Footprint" ""
-			(at 135.89 116.84 0)
-			(effects
-				(font
-					(size 1.27 1.27)
-				)
-				(hide yes)
-			)
-		)
-		(property "Datasheet" ""
-			(at 135.89 116.84 0)
-			(effects
-				(font
-					(size 1.27 1.27)
-				)
-				(hide yes)
-			)
-		)
-		(property "Description" "Power symbol creates a global label with name \"GND\" , ground"
-			(at 135.89 116.84 0)
-			(effects
-				(font
-					(size 1.27 1.27)
-				)
-				(hide yes)
-			)
-		)
-		(pin "1"
-		)
-		(instances
-			(project "board"
-				(path "/afefa398-9f39-4b22-97f8-dae9b102df0d/ed1ce839-173e-4775-a1bf-0525f06c4186"
-					(reference "#PWR0134")
-					(unit 1)
-				)
-			)
-		)
-	)
-	(symbol
-		(lib_id "power:GND")
 		(at 107.95 172.72 0)
 		(unit 1)
@@
 			)
 		)
-		(property "Footprint" ""
+		(property "Footprint" "Package_DIP:DIP-20_W7.62mm"
 			(at 107.95 152.4 0)
 			(effects
@@
 			)
 		)
-		(property "Footprint" ""
+		(property "Footprint" "Resistor_THT:R_Axial_DIN0207_L6.3mm_D2.5mm_P10.16mm_Horizontal"
 			(at 90.17 105.918 90)
 			(effects
@@
 			)
 		)
-		(property "Footprint" ""
+		(property "Footprint" "Resistor_THT:R_Axial_DIN0207_L6.3mm_D2.5mm_P10.16mm_Horizontal"
 			(at 128.27 103.378 90)
 			(effects
@@
 			)
 		)
-		(property "Footprint" ""
+		(property "Footprint" "Resistor_THT:R_Axial_DIN0207_L6.3mm_D2.5mm_P10.16mm_Horizontal"
 			(at 128.27 108.458 90)
 			(effects
@@
 			)
 		)
-		(property "Footprint" ""
+		(property "Footprint" "Package_DIP:DIP-20_W7.62mm"
 			(at 109.22 40.64 0)
 			(effects
@@
 			)
 		)
-		(property "Footprint" ""
+		(property "Footprint" "Resistor_THT:R_Axial_DIN0207_L6.3mm_D2.5mm_P10.16mm_Horizontal"
 			(at 90.17 113.538 90)
 			(effects
@@
 			)
 		)
-		(property "Footprint" ""
+		(property "Footprint" "Resistor_THT:R_Axial_DIN0207_L6.3mm_D2.5mm_P10.16mm_Horizontal"
 			(at 128.27 113.538 90)
 			(effects
@@
 	(symbol
 		(lib_id "power:+5V")
+		(at 78.74 87.63 0)
+		(unit 1)
+		(exclude_from_sim no)
+		(in_bom yes)
+		(on_board yes)
+		(dnp no)
+		(fields_autoplaced yes)
+		(property "Reference" "#PWR0127"
+			(at 78.74 91.44 0)
+			(effects
+				(font
+					(size 1.27 1.27)
+				)
+				(hide yes)
+			)
+		)
+		(property "Value" "+5V"
+			(at 78.74 82.55 0)
+			(effects
+				(font
+					(size 1.27 1.27)
+				)
+			)
+		)
+		(property "Footprint" ""
+			(at 78.74 87.63 0)
+			(effects
+				(font
+					(size 1.27 1.27)
+				)
+				(hide yes)
+			)
+		)
+		(property "Datasheet" ""
+			(at 78.74 87.63 0)
+			(effects
+				(font
+					(size 1.27 1.27)
+				)
+				(hide yes)
+			)
+		)
+		(property "Description" "Power symbol creates a global label with name \"+5V\""
+			(at 78.74 87.63 0)
+			(effects
+				(font
+					(size 1.27 1.27)
+				)
+				(hide yes)
+			)
+		)
+		(pin "1"
+		)
+		(instances
+			(project "board"
+				(path "/afefa398-9f39-4b22-97f8-dae9b102df0d/ed1ce839-173e-4775-a1bf-0525f06c4186"
+					(reference "#PWR0127")
+					(unit 1)
+				)
+			)
+		)
+	)
+	(symbol
+		(lib_id "power:+5V")
 		(at 109.22 20.32 0)
 		(unit 1)
@@
 	)
 	(symbol
+		(lib_id "power:+5V")
+		(at 135.89 87.63 0)
+		(unit 1)
+		(exclude_from_sim no)
+		(in_bom yes)
+		(on_board yes)
+		(dnp no)
+		(fields_autoplaced yes)
+		(property "Reference" "#PWR0134"
+			(at 135.89 91.44 0)
+			(effects
+				(font
+					(size 1.27 1.27)
+				)
+				(hide yes)
+			)
+		)
+		(property "Value" "+5V"
+			(at 135.89 82.55 0)
+			(effects
+				(font
+					(size 1.27 1.27)
+				)
+			)
+		)
+		(property "Footprint" ""
+			(at 135.89 87.63 0)
+			(effects
+				(font
+					(size 1.27 1.27)
+				)
+				(hide yes)
+			)
+		)
+		(property "Datasheet" ""
+			(at 135.89 87.63 0)
+			(effects
+				(font
+					(size 1.27 1.27)
+				)
+				(hide yes)
+			)
+		)
+		(property "Description" "Power symbol creates a global label with name \"+5V\""
+			(at 135.89 87.63 0)
+			(effects
+				(font
+					(size 1.27 1.27)
+				)
+				(hide yes)
+			)
+		)
+		(pin "1"
+		)
+		(instances
+			(project "board"
+				(path "/afefa398-9f39-4b22-97f8-dae9b102df0d/ed1ce839-173e-4775-a1bf-0525f06c4186"
+					(reference "#PWR0134")
+					(unit 1)
+				)
+			)
+		)
+	)
+	(symbol
 		(lib_id "Device:R")
 		(at 90.17 106.68 90)
@@
 			)
 		)
-		(property "Footprint" ""
+		(property "Footprint" "Resistor_THT:R_Axial_DIN0207_L6.3mm_D2.5mm_P10.16mm_Horizontal"
 			(at 90.17 108.458 90)
 			(effects
@@
 			)
 		)
-		(property "Footprint" ""
+		(property "Footprint" "Resistor_THT:R_Axial_DIN0207_L6.3mm_D2.5mm_P10.16mm_Horizontal"
 			(at 90.17 100.838 90)
 			(effects
@@
 	)
 	(symbol
-		(lib_id "power:GND")
-		(at 76.2 116.84 0)
-		(unit 1)
-		(exclude_from_sim no)
-		(in_bom yes)
-		(on_board yes)
-		(dnp no)
-		(fields_autoplaced yes)
-		(property "Reference" "#PWR0127"
-			(at 76.2 123.19 0)
-			(effects
-				(font
-					(size 1.27 1.27)
-				)
-				(hide yes)
-			)
-		)
-		(property "Value" "GND"
-			(at 76.2 121.92 0)
-			(effects
-				(font
-					(size 1.27 1.27)
-				)
-			)
-		)
-		(property "Footprint" ""
-			(at 76.2 116.84 0)
-			(effects
-				(font
-					(size 1.27 1.27)
-				)
-				(hide yes)
-			)
-		)
-		(property "Datasheet" ""
-			(at 76.2 116.84 0)
-			(effects
-				(font
-					(size 1.27 1.27)
-				)
-				(hide yes)
-			)
-		)
-		(property "Description" "Power symbol creates a global label with name \"GND\" , ground"
-			(at 76.2 116.84 0)
-			(effects
-				(font
-					(size 1.27 1.27)
-				)
-				(hide yes)
-			)
-		)
-		(pin "1"
-		)
-		(instances
-			(project "board"
-				(path "/afefa398-9f39-4b22-97f8-dae9b102df0d/ed1ce839-173e-4775-a1bf-0525f06c4186"
-					(reference "#PWR0127")
-					(unit 1)
-				)
-			)
-		)
-	)
-	(symbol
 		(lib_id "Device:R")
 		(at 90.17 93.98 90)
@@
 			)
 		)
-		(property "Footprint" ""
+		(property "Footprint" "Resistor_THT:R_Axial_DIN0207_L6.3mm_D2.5mm_P10.16mm_Horizontal"
 			(at 90.17 95.758 90)
 			(effects
@@
 			)
 		)
-		(property "Footprint" ""
+		(property "Footprint" "Capacitor_THT:C_Disc_D5.0mm_W2.5mm_P5.00mm"
 			(at 91.1352 186.69 0)
 			(effects
@@
 			)
 		)
-		(property "Footprint" ""
+		(property "Footprint" "Resistor_THT:R_Axial_DIN0207_L6.3mm_D2.5mm_P10.16mm_Horizontal"
 			(at 128.27 98.298 90)
 			(effects
@@
 			)
 		)
-		(property "Footprint" ""
+		(property "Footprint" "Resistor_THT:R_Axial_DIN0207_L6.3mm_D2.5mm_P10.16mm_Horizontal"
 			(at 90.17 98.298 90)
 			(effects
@@
 			)
 		)
-		(property "Footprint" ""
+		(property "Footprint" "Resistor_THT:R_Axial_DIN0207_L6.3mm_D2.5mm_P10.16mm_Horizontal"
 			(at 128.27 100.838 90)
 			(effects
@@
 			)
 		)
-		(property "Footprint" ""
+		(property "Footprint" "Resistor_THT:R_Axial_DIN0207_L6.3mm_D2.5mm_P10.16mm_Horizontal"
 			(at 90.17 103.378 90)
 			(effects
@@
 			)
 		)
-		(property "Footprint" ""
+		(property "Footprint" "Resistor_THT:R_Axial_DIN0207_L6.3mm_D2.5mm_P10.16mm_Horizontal"
 			(at 128.27 105.918 90)
 			(effects
@@
 			)
 		)
-		(property "Footprint" ""
+		(property "Footprint" "Capacitor_THT:C_Disc_D5.0mm_W2.5mm_P5.00mm"
 			(at 69.5452 52.07 0)
 			(effects
@@
 			)
 		)
-		(property "Footprint" ""
+		(property "Footprint" "Resistor_THT:R_Axial_DIN0207_L6.3mm_D2.5mm_P10.16mm_Horizontal"
 			(at 128.27 95.758 90)
 			(effects

Commit message: checkpoint
Parts:
- removed R17, R18, R19, R20, R21, R22, R23, R24, R25, R26, R27, R28, R29, R30, R31, R32: 330, Resistor_THT:R_Axial_DIN0207_L6.3mm_D2.5mm_P10.16mm_Horizontal, symbol Device:R
- added RN1, RN2: 330, Package_DIP:DIP-16_W7.62mm, symbol Device:R_Pack08
Connections:
- net +5V: now also U24.13 (DIG2_CA), U24.14 (DIG1_CA); no longer U24.4 (DP1), U24.9 (DP2)
- net at U23.2 (O0): now also RN1.2 (R2.1)
- net at U24.16 (DIG1_A): now also RN1.15 (R2.2)
- net at U24.11 (DIG2_A): now also RN2.2 (R2.1)
- net at U22.2 (O0): now also RN2.16 (R1.2)
- net at U22.12 (O4): now also RN2.10 (R7.2)
- net at U22.15 (O5): now also RN2.13 (R4.2)
- net at U22.16 (O6): now also RN2.12 (R5.2)
- net at U22.19 (O7): now also RN2.15 (R2.2)
- net at U22.5 (O1): now also RN2.14 (R3.2)
- net at U22.6 (O2): now also RN2.11 (R6.2)
- net at U22.9 (O3): now also RN2.9 (R8.2)
- net at U23.15 (O5): now also RN1.3 (R3.1)
- net at U24.18 (DIG1_F): now also RN1.13 (R4.2)
- net at U24.5 (DIG2_E): now also RN2.8 (R8.1)
- net at U24.7 (DIG2_G): now also RN2.6 (R6.1)
- net at U23.12 (O4): now also RN1.8 (R8.1)
- net at U23.16 (O6): now also RN1.6 (R6.1)
- net at U23.19 (O7): now also RN1.1 (R1.1)
- net at U23.5 (O1): now also RN1.4 (R4.1)
- net at U23.6 (O2): now also RN1.5 (R5.1)
- net at U23.9 (O3): now also RN1.7 (R7.1)
- net at U24.17 (DIG1_G): now also RN1.14 (R3.2)
- net at U24.2 (DIG1_D): now also RN1.11 (R6.2)
- net at U24.15 (DIG1_B): now also RN1.16 (R1.2)
- net at U24.8 (DIG2_C): now also RN2.5 (R5.1)
- net at U24.3 (DIG1_C): now also RN1.10 (R7.2)
- net at U24.6 (DIG2_D): now also RN2.7 (R7.1)
- net at U24.1 (DIG1_E): now also RN1.12 (R5.2)
- net at U24.10 (DIG2_B): now also RN2.3 (R3.1)
- net at U24.12 (DIG2_F): now also RN2.1 (R1.1)
- new net: RN1.9 (R8.2), U24.4 (DP1)
- new net: RN2.4 (R4.1), U24.9 (DP2)
Other:
- moved on the sheet: C36, C37, U22, U23, U24

Commit message: checkpoint
Parts:
- RN1, RN2: digikey (none) -> https://www.digikey.com/en/products/detail/bourns-inc/4116R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
Changed lines of the file:
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@@
+			)
+		)
+		(property "digikey" "https://www.digikey.com/en/products/detail/bourns-inc/4116R-R2R-103LF/2565166"
+			(at 82.55 91.44 90)
+			(effects
+				(font
+					(size 1.27 1.27)
+				)
+				(hide yes)
 			)
 		)
@@
 			(effects
 				(font
+					(size 1.27 1.27)
+				)
+				(hide yes)
+			)
+		)
+		(property "digikey" "https://www.digikey.com/en/products/detail/bourns-inc/4116R-R2R-103LF/2565166"
+			(at 199.39 92.71 90)
+			(effects
+				(font

Commit message: checkpoint
Parts:
- removed C37: 100nF, Capacitor_THT:C_Disc_D5.0mm_W2.5mm_P5.00mm, symbol Device:C
- removed RN1, RN2: 330, Package_DIP:DIP-16_W7.62mm, symbol Device:R_Pack08
- removed U22: 74HC373, Package_DIP:DIP-20_W7.62mm, symbol 74xx:74HC373
- removed U24: DA56-11SRWA, Display_7Segment:DA56-11SURKWA, symbol Display_Character:DA56-11SRWA
- added C24: 100nF, Capacitor_THT:C_Disc_D5.0mm_W2.5mm_P5.00mm, symbol Device:C
- added C25: 10nF, Capacitor_THT:C_Disc_D3.0mm_W1.6mm_P2.50mm, symbol Device:C
- added C26: 100µF, Capacitor_THT:CP_Radial_D5.0mm_P2.50mm, symbol Device:C
- added J7: STEREO_OUT, board:SAMESKY_SJ3-35063B, symbol SS_AUDIO:SJ3-35063B
- added LS1: Speaker, Buzzer_Beeper:MagneticBuzzer_StarMicronics_QMX, symbol Device:Speaker
- added R52, R53: 1K, Resistor_THT:R_Axial_DIN0207_L6.3mm_D2.5mm_P10.16mm_Horizontal, symbol Device:R
- added R57, R58: 100, Resistor_THT:R_Axial_DIN0207_L6.3mm_D2.5mm_P10.16mm_Horizontal, symbol Device:R
- added R59: 47, Resistor_THT:R_Axial_DIN0207_L6.3mm_D2.5mm_P10.16mm_Horizontal, symbol Device:R
- added R60: 4610X-R2R-103LF, board:BO_4610X, symbol 68k_board:4610X-R2R-103LF
- added U15: LM358, Package_DIP:DIP-8_W7.62mm, symbol Amplifier_Operational:LM358
Connections:
- net +5V: now also C24.1, U15.8 (V+)
- net GND: now also C24.2, C25.2, J7.1, LS1.2, R53.1, R60.10, U15.4 (V-), U15.5 (+)
- net AUDIO4: now reaches U23.12 (O4)
- net AUDIO4: now also R60.5
- net AUDIO5: now reaches U23.15 (O5)
- net AUDIO5: now also R60.4
- net AUDIO6: now reaches U23.16 (O6)
- net AUDIO6: now also R60.3
- net AUDIO7: now reaches U23.19 (O7)
- net AUDIO7: now also R60.2
- net AUDIO0: now reaches U23.2 (O0)
- net AUDIO0: now also R60.9
- net AUDIO1: now reaches U23.5 (O1)
- net AUDIO1: now also R60.8
- net AUDIO2: now reaches U23.6 (O2)
- net AUDIO2: now also R60.7
- net AUDIO3: now reaches U23.9 (O3)
- net AUDIO3: now also R60.6
- net DBGHILED_LE renamed AUDIO_LE
- new net: LS1.1, R59.1
- new net: J7.4, R59.2
- new net: C25.1, C26.1, R52.2
- new net: C26.2, R53.2, R57.2, R58.2
- new net: U15.6 (-), U15.7
- new net: J7.2, R57.1
- new net: J7.3, R58.1
- new net: R60.1, U15.3 (+)
- new net: R52.1, U15.1, U15.2 (-)
Other:
- moved on the sheet: C36
