File: board/board.kicad_sch (KiCad schematic)
At the start: 0 parts

Commit message: checkpoint - maybe unfinishable
Changed lines of the file:
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@@
 	(paper "A4")
 	(sheet
-		(at 127 72.39)
-		(size 50.8 24.13)
+		(at 88.9 63.5)
+		(size 40 20)
 		(exclude_from_sim no)
 		(in_bom yes)
@@
 		)
 		(property "Sheetname" "GLUE"
-			(at 127 71.6784 0)
+			(at 88.9 62.7884 0)
 			(effects
 				(font
@@
 		)
 		(property "Sheetfile" "glue.kicad_sch"
-			(at 127 97.1046 0)
+			(at 88.9 88.2146 0)
 			(effects
 				(font
@@
 	)
 	(sheet
-		(at 130.81 115.57)
-		(size 49.53 26.67)
+		(at 88.9 101.6)
+		(size 40 20)
 		(exclude_from_sim no)
 		(in_bom yes)
@@
 		)
 		(property "Sheetname" "COMPOSITE"
-			(at 130.81 114.8584 0)
+			(at 88.9 100.8884 0)
 			(effects
 				(font
@@
 		)
 		(property "Sheetfile" "composite.kicad_sch"
-			(at 130.81 142.8246 0)
+			(at 88.9 128.8546 0)
 			(effects
 				(font
@@
 	)
 	(sheet
-		(at 45.72 119.38)
-		(size 46.99 39.37)
+		(at 25.4 101.6)
+		(size 40 20)
 		(exclude_from_sim no)
 		(in_bom yes)
@@
 		)
 		(property "Sheetname" "ROM"
-			(at 45.72 118.6684 0)
+			(at 25.4 100.8884 0)
 			(effects
 				(font
@@
 		)
 		(property "Sheetfile" "rom.kicad_sch"
-			(at 45.72 159.3346 0)
+			(at 25.4 141.5546 0)
 			(effects
 				(font
@@
 	)
 	(sheet
-		(at 29.21 26.67)
-		(size 43.18 20.32)
+		(at 25.4 25.4)
+		(size 40 20)
 		(exclude_from_sim no)
 		(in_bom yes)
@@
 		)
 		(property "Sheetname" "POWER_CLOCK"
-			(at 29.21 25.9584 0)
+			(at 25.4 24.6884 0)
 			(effects
 				(font
@@
 		)
 		(property "Sheetfile" "power-clock.kicad_sch"
-			(at 29.21 47.5746 0)
+			(at 25.4 46.3046 0)
 			(effects
 				(font
@@
 	)
 	(sheet
-		(at 195.58 48.26)
-		(size 40.64 20.32)
+		(at 152.4 25.4)
+		(size 40 20)
 		(exclude_from_sim no)
 		(in_bom yes)
@@
 		)
 		(property "Sheetname" "IO"
-			(at 195.58 47.5484 0)
+			(at 152.4 24.6884 0)
 			(effects
 				(font
@@
 		)
 		(property "Sheetfile" "io.kicad_sch"
-			(at 195.58 69.1646 0)
+			(at 152.4 46.3046 0)
 			(effects
 				(font
@@
 	)
 	(sheet
-		(at 21.59 52.07)
-		(size 45.72 22.86)
+		(at 152.4 101.6)
+		(size 40 20)
 		(exclude_from_sim no)
 		(in_bom yes)
@@
 		)
 		(property "Sheetname" "EXPANSION_BUS"
-			(at 21.59 51.3584 0)
+			(at 152.4 100.8884 0)
 			(effects
 				(font
@@
 		)
 		(property "Sheetfile" "expansion.kicad_sch"
-			(at 21.59 75.5146 0)
+			(at 152.4 125.0446 0)
 			(effects
 				(font
@@
 	)
 	(sheet
-		(at 127 25.4)
-		(size 40.64 19.05)
+		(at 88.9 25.4)
+		(size 40 20)
 		(exclude_from_sim no)
 		(in_bom yes)
@@
 		)
 		(property "Sheetname" "RAM"
-			(at 127 24.6884 0)
+			(at 88.9 24.6884 0)
 			(effects
 				(font
@@
 		)
 		(property "Sheetfile" "ram.kicad_sch"
-			(at 127 45.0346 0)
+			(at 88.9 45.0346 0)
 			(effects
 				(font
@@
 	)
 	(sheet
-		(at 41.91 81.28)
-		(size 48.26 20.32)
+		(at 25.4 63.5)
+		(size 40 20)
 		(exclude_from_sim no)
 		(in_bom yes)
@@
 		)
 		(property "Sheetname" "CPU"
-			(at 41.91 80.5684 0)
+			(at 25.4 62.7884 0)
 			(effects
 				(font
@@
 		)
 		(property "Sheetfile" "cpu.kicad_sch"
-			(at 41.91 102.1846 0)
+			(at 25.4 84.4046 0)
 			(effects
 				(font
@@
 	)
 	(sheet
-		(at 199.39 81.28)
-		(size 39.37 24.13)
+		(at 152.4 63.5)
+		(size 40 20)
 		(exclude_from_sim no)
 		(in_bom yes)
@@
 		)
 		(property "Sheetname" "DEBUG_LED"
-			(at 199.39 80.5684 0)
+			(at 152.4 62.7884 0)
 			(effects
 				(font
@@
 		)
 		(property "Sheetfile" "debug-led.kicad_sch"
-			(at 199.39 105.9946 0)
-			(effects
-				(font
+			(at 152.4 88.2146 0)
+			(effects
+				(font

Commit message: checkpoint before deleting composite video
Other:
- sheet COMPOSITE renamed ONBOARDVID
Changed lines of the file:
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@@
 			(color 0 0 0 0.0000)
 		)
-		(property "Sheetname" "COMPOSITE"
+		(property "Sheetname" "ONBOARDVID"
 			(at 88.9 100.8884 0)
 			(effects

Commit message: checkpoint
Other:
- sheet DEBUG_LED renamed AUDIO
- sheet EXPANSION_BUS renamed APP_ENGINE
- added sheet TESTPOINTS (test-points.kicad_sch)
Changed lines of the file:
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@@
 		(on_board yes)
 		(dnp no)
-		(fields_autoplaced yes)
 		(stroke
 			(width 0.1524)
@@
 		)
 		(property "Sheetfile" "rom.kicad_sch"
-			(at 25.4 141.5546 0)
+			(at 25.654 122.936 0)
 			(effects
 				(font
@@
 			(color 0 0 0 0.0000)
 		)
-		(property "Sheetname" "EXPANSION_BUS"
+		(property "Sheetname" "APP_ENGINE"
 			(at 152.4 100.8884 0)
 			(effects
@@
 	)
 	(sheet
+		(at 25.4 138.43)
+		(size 40.64 20.32)
+		(exclude_from_sim no)
+		(in_bom yes)
+		(on_board yes)
+		(dnp no)
+		(fields_autoplaced yes)
+		(stroke
+			(width 0.1524)
+			(type solid)
+		)
+		(fill
+			(color 0 0 0 0.0000)
+		)
+		(property "Sheetname" "TESTPOINTS"
+			(at 25.4 137.7184 0)
+			(effects
+				(font
+					(size 1.27 1.27)
+				)
+				(justify left bottom)
+			)
+		)
+		(property "Sheetfile" "test-points.kicad_sch"
+			(at 25.4 159.3346 0)
+			(effects
+				(font
+					(size 1.27 1.27)
+				)
+				(justify left top)
+			)
+		)
+		(instances
+			(project "board"
+				(path "/afefa398-9f39-4b22-97f8-dae9b102df0d"
+					(page "11")
+				)
+			)
+		)
+	)
+	(sheet
 		(at 88.9 25.4)
 		(size 40 20)
@@
 			(color 0 0 0 0.0000)
 		)
-		(property "Sheetname" "DEBUG_LED"
+		(property "Sheetname" "AUDIO"
 			(at 152.4 62.7884 0)
 			(effects

Commit message: Board rev1 PCB complete, already have a spot fix
Other:
- added sheet COMPACT_FLASH (compact-flash.kicad_sch)
Changed lines of the file:
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@@
+	)
+	(sheet
+		(at 88.9 138.43)
+		(size 40.64 20.32)
+		(exclude_from_sim no)
+		(in_bom yes)
+		(on_board yes)
+		(dnp no)
+		(fields_autoplaced yes)
+		(stroke
+			(width 0.1524)
+			(type solid)
+		)
+		(fill
+			(color 0 0 0 0.0000)
+		)
+		(property "Sheetname" "COMPACT_FLASH"
+			(at 88.9 137.7184 0)
+			(effects
+				(font
+					(size 1.27 1.27)
+				)
+				(justify left bottom)
+			)
+		)
+		(property "Sheetfile" "compact-flash.kicad_sch"
+			(at 88.9 159.3346 0)
+			(effects
+				(font
+					(size 1.27 1.27)
+				)
+				(justify left top)
+			)
+		)
+		(instances
+			(project "board"
+				(path "/afefa398-9f39-4b22-97f8-dae9b102df0d"
+					(page "12")
+				)
+			)
+		)
 	)
 	(sheet
